Commit message: Update robot model dimensions and file references

File: src/glados_description/models/glados/model_test.urdf (robot description, URDF)
Before this commit: robot glados, 6 links, 5 joints
Links:
- link base_link: geometry collision box size=0.65 0.245 0.175; visual box size=0.65 0.245 0.175
- link front_left_wheel: geometry collision sphere radius=0.1; visual mesh filename=package://glados_description/models/glados/meshes/mecanum_w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 scale=0.006 0.006 0.006
- link front_right_wheel: geometry collision sphere radius=0.1; visual mesh filename=package://glados_description/models/glados/meshes/mecanum_w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 scale=0.006 0.006 0.006
- link rear_left_wheel: geometry collision sphere radius=0.1; visual mesh filename=package://glados_description/models/glados/meshes/mecanum_w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 scale=0.006 0.006 0.006
- link rear_right_wheel: geometry collision sphere radius=0.1; visual mesh filename=package://glados_description/models/glados/meshes/mecanum_w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 scale=0.006 0.006 0.006

Commit message: Update SDF and URDF models for improved robot configuration

File: src/glados_description/models/glados/model_test.urdf (robot description, URDF)
Before this commit: robot glados, 6 links, 5 joints
Links:
- link front_left_wheel: geometry collision sphere radius=0.1; visual mesh filename=package://glados_description/models/glados/meshes/mecanum_w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 scale=0.00 0.001 0.001
- link front_right_wheel: geometry collision sphere radius=0.1; visual mesh filename=package://glados_description/models/glados/meshes/mecanum_w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 scale=0.00 0.001 0.001
- link rear_left_wheel: geometry collision sphere radius=0.1; visual mesh filename=package://glados_description/models/glados/meshes/mecanum_w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 scale=0.00 0.001 0.001
- link rear_right_wheel: geometry collision sphere radius=0.1; visual mesh filename=package://glados_description/models/glados/meshes/mecanum_w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 scale=0.00 0.001 0.001
Joints:
- joint front_left_wheel_joint: origin xyz=0.554283 0.625029 0 rpy=-1.5707963267948966 0 0 -> xyz=0.20 0.01225 0 rpy=-1.5707963267948966 0 0
- joint front_right_wheel_joint: origin xyz=0.554282 -0.625029 0 rpy=-1.5707963267948966 0 0 -> xyz=0.20 -0.01225 0 rpy=-1.5707963267948966 0 0
- joint rear_left_wheel_joint: origin xyz=-0.957138 0.625029 0 rpy=-1.5707963267948966 0 0 -> xyz=-0.20 0.01225 0 rpy=-1.5707963267948966 0 0
- joint rear_right_wheel_joint: origin xyz=-0.957138 -0.625029 0 rpy=-1.5707963267948966 0 0 -> xyz=-0.20 -0.01225 0 rpy=-1.5707963267948966 0 0
