Commit message: urdf model

File: src/glados_description/models/glados/model.urdf (robot description, URDF)
Before this commit: robot glados, 8 links, 7 joints
Links:
- link base_footprint: geometry 
- link camera_link: mass 0.1 -> None; geometry visual mesh filename=package://glados_description/models/glados/meshes/realsense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
- link front_left_wheel: mass 2 -> None; geometry visual mesh filename=package://glados_description/models/glados/meshes/mecanum_w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 scale=0.002 0.002 0.002
- link front_right_wheel: mass 2 -> None; geometry visual mesh filename=package://glados_description/models/glados/meshes/mecanum_w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 scale=0.002 0.002 0.002
- link lidar_link: mass 0.1 -> None; geometry visual cylinder length=0.04 radius=0.04
- link rear_left_wheel: mass 2 -> None; geometry visual mesh filename=package://glados_description/models/glados/meshes/mecanum_w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 scale=0.002 0.002 0.002
- link rear_right_wheel: mass 2 -> None; geometry visual mesh filename=package://glados_description/models/glados/meshes/mecanum_w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 scale=0.002 0.002 0.002
Joints:
- removed joint camera_joint
- added joint chassis_to_camera: type fixed, parent chassis, child camera_link, origin xyz=0.330 0 -0.0125 rpy=0 0 0
- joint front_left_wheel_joint: limit (none) -> lower=-1.79769e+308 upper=1.79769e+308 effort=0 velocity=0; type continuous -> revolute
- joint front_right_wheel_joint: limit (none) -> lower=-1.79769e+308 upper=1.79769e+308 effort=0 velocity=0; type continuous -> revolute
- joint rear_left_wheel_joint: limit (none) -> lower=-1.79769e+308 upper=1.79769e+308 effort=0 velocity=0; type continuous -> revolute
- joint rear_right_wheel_joint: limit (none) -> lower=-1.79769e+308 upper=1.79769e+308 effort=0 velocity=0; type continuous -> revolute

Commit message: added ros realsense package and realsense lib v456 install in docker

File: src/glados_description/models/glados/model.urdf (robot description, URDF)
Before this commit: robot glados, 8 links, 7 joints
Links:
- added link top_box; collision box size=0.18 0.245 0.18; visual box size=0.18 0.245 0.18
Joints:
- added joint chassis_to_top_box: type fixed, parent chassis, child top_box, origin xyz=-0.12 0 0.025 rpy=0 0 0

Commit message: aruco markers and nav2 configuration

File: src/glados_description/models/glados/model.urdf (robot description, URDF)
Before this commit: robot glados, 9 links, 8 joints
Links:
- removed link top_box
- added link battery; collision box size=0.18 0.245 0.18; visual box size=0.18 0.245 0.18
- added link front_left_pillar; collision box size=0.18 0.01 0.01; visual box size=0.18 0.01 0.01
- added link front_right_pillar; collision box size=0.18 0.01 0.01; visual box size=0.18 0.01 0.01
- added link roof; collision box size=0.535 0.245 0.01; visual box size=0.535 0.245 0.01
Joints:
- removed joint chassis_to_top_box
- added joint chassis_to_battery: type fixed, parent chassis, child battery, origin xyz=-0.12 0 0.115 rpy=0 0 0
- added joint front_left_pillar_to_chassis: type fixed, parent chassis, child front_left_pillar, origin xyz=0.32 0.1175 0.025 rpy=0 -1.57 0
- added joint front_right_pillar_to_chassis: type fixed, parent chassis, child front_right_pillar, origin xyz=0.32 -0.1175 0.025 rpy=0 -1.57 0
- added joint roof_to_chassis: type fixed, parent chassis, child roof, origin xyz=0.0575 0 0.21 rpy=0 0 0
- joint chassis_to_camera: origin xyz=0.330 0 -0.0125 rpy=0 0 0 -> xyz=0.305 0 0.195 rpy=0 0 0
- joint front_left_wheel_joint: axis 0 0 1 -> 0 1 0; origin xyz=0.2 0.1625 0 rpy=-1.5707 0 0 -> xyz=0.2 0.1635 0 rpy=0 0 0
- joint front_right_wheel_joint: axis 0 0 1 -> 0 1 0; origin xyz=0.2 -0.1625 0 rpy=-1.5707 0 0 -> xyz=0.2 -0.1635 0 rpy=0 0 0
- joint lidar_joint: origin xyz=0.325 0 0.045 rpy=0 0 0 -> xyz=0.245 0 0.23 rpy=0 0 0
- joint rear_left_wheel_joint: axis 0 0 1 -> 0 1 0; origin xyz=-0.2 0.1625 0 rpy=-1.5707 0 0 -> xyz=-0.2 0.1635 0 rpy=0 0 0
- joint rear_right_wheel_joint: axis 0 0 1 -> 0 1 0; origin xyz=-0.2 -0.1625 0 rpy=-1.5707 0 0 -> xyz=-0.2 -0.1635 0 rpy=0 0 0
